File: kicad/mc60.sch (KiCad schematic (older format))
At the start: 1 part

Commit message: schematic wip
Parts:
- added J?: SIM_Card, symbol mc60_library:SIM_Card
- added SD?: SD_CARD_Micro, symbol haathi:SD_CARD_Micro
Other:
- moved on the sheet: U?
Changed lines of the file:
@@
 EESchema Schematic File Version 4
+LIBS:mc60-cache
 EELAYER 26 0
 EELAYER END
@@
 L mc60_library:MC60_0 U?
 U 1 1 5ACB0259
-P 8000 5100
-F 0 "U?" H 8000 6925 60  0000 C CNB
-F 1 "MC60_0" H 8000 6825 60  0000 C CNB
-F 2 "XCVR_MC60" H 8000 4850 60  0001 C BNB
-F 3 "MC60" H 8000 5350 60  0001 C BNB
-	1    8000 5100
+P 3550 3300
+F 0 "U?" H 3550 5125 60  0000 C CNB
+F 1 "MC60_0" H 3550 5025 60  0000 C CNB
+F 2 "XCVR_MC60" H 3550 3050 60  0001 C BNB
+F 3 "MC60" H 3550 3550 60  0001 C BNB
+	1    3550 3300
 	1    0    0    -1
 $EndComp
+$Comp
+L haathi:SD_CARD_Micro SD?
+U 1 1 5ACB96AA
+P 7650 2900
+F 0 "SD?" H 8050 3525 60  0000 C CNN
+F 1 "SD_CARD_Micro" H 8050 3425 60  0000 C CNN
+F 2 "" H 7550 2900 60  0000 C CNN
+F 3 "" H 7550 2900 60  0000 C CNN
+	1    7650 2900
+	1    0    0    -1
+$EndComp
+$Comp
+L mc60_library:SIM_Card J?
+U 1 1 5ACBF9E1
+P 8050 3725
+F 0 "J?" H 8500 3875 50  0000 L CNN
+F 1 "SIM_Card" H 8500 3775 50  0000 L CNN
+F 2 "" H 8050 4075 50  0000 C CNN
+F 3 "" H 8000 3725 50  0000 C CNN
+	1    8050 3725
+	1    0    0    -1
+$EndComp

Commit message: schematic wip
Parts:
- added AE?: Antenna_BT, symbol mc60_library:Antenna_Chip
- added C? (x4): 33pF, symbol mc60_library:C_NP
- added CN?: Conn_GPS, symbol mc60_library:Conn_Coaxial
- added CN?: Conn_GNSS, symbol mc60_library:Conn_Coaxial
- added R? (x2): 100k, symbol mc60_library:R
- added R? (x3): 22E, symbol mc60_library:R
- added R?: 0E, symbol mc60_library:R
- CN?: renamed from SD?; value SD_CARD_Micro -> SD_CARD
- gave numbers to parts that had none: 1
Connections:
- net labels added: ANT_BT, ANT_GNSS, ANT_GPS, BT, GND, SD_CLK, SD_CMD, SD_DAT, SD_DET, SIM1_VDD, SIM_CLK, SIM_DAT, SIM_RST, VCC, VDD_EXT
- wire segments 0 -> 73
- no-connect marks 0 -> 9
Other:
- moved on the sheet: CN?

Commit message: schematic wip
Parts:
- added D?: Diode_TVS, symbol mc60_library:Diode_TVS
- added D? (x3): LED, symbol mc60_library:LED
- added Q? (x3): DTC114E, symbol mc60_library:DTC114E
- added R? (x3): 100k, symbol mc60_library:R
- CN?: symbol haathi:SD_CARD_Micro -> mc60_library:SD_CARD_Micro; manf# (none) -> mfr_pn
Connections:
- net labels added: 1PPS, GNSSVCC, NETLIGHT, PWRKEY, RST, VBAT
- wire segments 73 -> 140
- no-connect marks 9 -> 11
Other:
- note added: "Route to SIM_GND seperately"
- moved on the sheet: AE?, CN?, R?

Commit message: schematic wip
Parts:
- removed R?: 100k, symbol mc60_library:R
- added C? (x3): 470uF, symbol mc60_library:C_POL
- added C? (x4): 100nF, symbol mc60_library:C_NP
- added C?: 100uF, symbol mc60_library:C_POL
- added C?: 4u7, symbol mc60_library:C_POL
- added C?: 33pF, symbol mc60_library:C_NP
- added C?: 10pF, symbol mc60_library:C_NP
- added Q?: DTC114E, symbol mc60_library:DTC143
- added R?: 51k, symbol mc60_library:R
- added R?: 124k, symbol mc60_library:R
- added R?: 56k, symbol mc60_library:R
- added R?: 470, symbol mc60_library:R
- added R?: 47k, symbol mc60_library:R
- added U?: MIC29302, Package_TO_SOT_SMD:TO-252-6, symbol mc60_library:MIC29302
- added U?: LP5907, Package_TO_SOT_SMD:TO-252-6, symbol mc60_library:LP5907
- R? (x2): value 100k -> 470
Connections:
- net labels added: GNSS_VCC_EN, GSM_PWR_EN, VIN
- wire segments 140 -> 222
Other:
- moved on the sheet: D?, Q?, R?

Commit message: schematic wip
Parts:
- removed D?: LED, symbol mc60_library:LED
- removed R?: 0E, symbol mc60_library:R
- added C1, C37, C42: 4u7, symbol mc60_library:C_POL
- added C12, C15, C26, C43: 10uF, symbol mc60_library:C_POL
- added C13, C18, C20, C22, C24: 33pF, symbol mc60_library:C_NP
- added C14, C19, C21, C23, C25: 10pF, symbol mc60_library:C_NP
- added C16, C17, C41, C44: 100nF, symbol mc60_library:C_NP
- added C2, C3, C4, C5, C6, C7: 10pF_DNP, symbol mc60_library:C_NP
- added C31: 1uF, symbol mc60_library:C_NP
- added C40: 100uF, symbol mc60_library:C_POL
- added CN5: Audio-Jack-4, symbol mc60_library:Audio-Jack-4
- added CN6: UART_DBG, symbol mc60_library:Conn_01x03
- added CN7: CONTROL, symbol mc60_library:CONN_01X08
- added CN8: UART, symbol mc60_library:CONN_01X08
- added D1: Diode_TVS, symbol mc60_library:Diode_TVS
- added D5, D6: ESD9B5.0ST5G, symbol mc60_library:Diode_TVS_1
- added D7: 5V1/1W, symbol mc60_library:diode_zener
- added D8: LED, symbol mc60_library:LED
- added J1: B_LS_N, symbol mc60_library:Conn_01x01
- added J2: B_VRTC, symbol mc60_library:Conn_01x01
- added J3: B_SPKP, symbol mc60_library:Conn_01x01
- added J4: B_SPKN, symbol mc60_library:Conn_01x01
- added J5: B_ADC, symbol mc60_library:Conn_01x01
- added JP1: 3V3_EXT<>5V, symbol mc60_library:SolderJumper_3_Open
- added JP2: GSM_PWR_EN, symbol mc60_library:SolderJumper_3_Open
- added R11, R12, R13, R15, R2, R3, R4: 0E, symbol mc60_library:R
- added R14: 10k, symbol mc60_library:R
- added S1: SW-ON, symbol dh:SW-SPST-M
- added U2: TXB0108PWR, Package_TO_SOT_SMD:USON-20_2x4mm_P0.4mm, symbol mc60_library:TXB0108PWR
- added U5: LP5907-2V8, Package_TO_SOT_SMD:TO-252-6, symbol mc60_library:LP5907
- AE1: renamed from AE?; value Antenna_BT -> ANT_BT
- C38: renamed from C?; value 4u7 -> 10uF
- R18: renamed from R?; value 470 -> 300E
- R8, R9: renamed from R?; value 470 -> 470E
- U4: renamed from U?; value LP5907 -> LP5907-3V3
- gave numbers to parts that had none: 36
Connections:
- net labels added: 2V8_SD, 3V3_EXT, 5V, ADC, CTS, CTS>, DBG_RXD, DBG_TXD, DCD, DCD>, DTR, DTR>, GNDD, GNDREF, GND_REF, LEFT, LOUD_SPKP, MIC+, MIC-, RIGHT, RING, RING>, RTS, RTS>, RXD, RXD>, SD_DET>, SIM_GND, SPKN, SPKP, TXD, TXD>, VCCB, VDD
- net labels removed: BT, VCC, VIN
- wire segments 222 -> 467
- no-connect marks 11 -> 17
Other:
- note added: "2V8,20mA max."
- note added: "ANTENNAE"
- note added: "AUDIO"
- note added: "CITA STYLE\nCONNECTION"
- note added: "CONTROLS"
- note added: "HEADERS"
- note added: "NEAR GNSSVCC PIN"
- note added: "NEAR SD-CARD"
- note added: "NEAR VBAT PINS"
- note added: "PLACE NEAR MC60 PINS"
- note added: "POWER SUPPLY"
- note added: "Route to MC60 SIM_GND seperately"
- note added: "SD_CARD"
- note added: "SIM_CARD"
- note added: "UART LEVEL TRANSLATION"
- note removed: "Route to SIM_GND seperately"
- moved on the sheet: AE1, C10, C11, C28, C32, C33, C34, C36, C39, C8, C9, CN1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

Commit message: schematic WIP
Parts:
- AE1: manf# (none) -> SR4W035
- CN5: manf# (none) -> SJ-43514-SMT-TR
- D1, D4: value Diode_TVS -> RClamp0854P.TCT
- D2: value LED -> LED_NET
- D3: value LED -> LED_FIX
- D8: value LED -> LED_PWR
- renumbered CN6 to H1, CN8 to H2, CN7 to H3
Connections:
- net labels added: LOUD_SPKN, RXD_AUX, RXD_G, TXD_AUX, TXD_G, VRTC
- wire segments 467 -> 468
Other:
- note added: "2V8 for SD-CARD"
- note added: "3V3 for GNSS DOMAIN"
- note added: "4V for GPS DOMAIN"
- note added: "5V/3A (2A min)"
- note added: "AUDIO - EXT. EARPHONE/MIC"
- note added: "CITA STYLE\nTRRS\nCONNECTION"
- note added: "INDICATORS - CONTROLS"
- note added: "JP2 > 5V = OFF (VReg U3 is disabled).\nJP2 > GND = ON (VReg U3 is enabled).\n"
- note added: "LED flashes at 1pps\nafter GPS fix"
- note added: "LED flashes\nindicate Network status"
- note added: "Power control\nPush S1 for ON, Push S1 for OFF\nOR via external "RST" signal"
- note added: "Reference design does not have SD-Card\nmikroe.de "click" uses VDD_EXT which is limited to 20mA max\nSome SD-Cards require up to 100mA during Write cycles"
- note added: "UART output voltage can be either\n5V (derived from main input) or\n3V3 (derived from external input)"
- note removed: "AUDIO"
- note removed: "CITA STYLE\nCONNECTION"
- note removed: "CONTROLS"
- moved on the sheet: D2, D3, D8, Q1, Q2, R12, R13, R19, R20, R8, R9

Commit message: schematic wip
Parts:
- C1, C12, C15, C26, C37, C38, C42, C43: footprint (none) -> Capacitors_SMD:C_0805
- C10, C11, C13, C14, C16, C17, C18, C19, C2, C20, C21, C22, C23, C24, C25, C28, C3, C31, C32, C33, C34, C36, C39, C4, C41, C44, C5, C6, C7, C8, C9, R1, R10, R11, R12, R13, R14, R15, R16, R17, R19, R2, R20, R3, R4, R5, R6, R7: footprint (none) -> Capacitors_SMD:C_0603
- D7: value 5V1/1W -> PDZVTR5.1B
- R18: value 300E -> 390E; footprint (none) -> Capacitors_SMD:C_0603
- R8: value 470E -> 390E; footprint (none) -> Capacitors_SMD:C_0603
- R9: value 470E -> 270E; footprint (none) -> Capacitors_SMD:C_0603
- S1: symbol dh:SW-SPST-M -> mc60_library:SW-SPST-M; manf# (none) -> mfr_pn
- U1: footprint XCVR_MC60 -> (none)
Other:
- moved on the sheet: C10, C11, C8, C9, CN3, CN4, D1, D4, R1, R10, R5, R6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

Commit message: schematic WIP
Parts:
- AE1: footprint (none) -> mc60_fp:ant_bt_inpaq5036
- C1, C12, C15, C26, C37, C38, C42, C43: footprint Capacitors_SMD:C_0805 -> mc60_fp:C_0805
- C10, C11, C13, C14, C16, C17, C18, C19, C2, C20, C21, C22, C23, C24, C25, C28, C3, C31, C32, C33, C34, C36, C39, C4, C41, C44, C5, C6, C7, C8, C9: footprint Capacitors_SMD:C_0603 -> mc60_fp:C_0603
- C27, C29, C30: footprint (none) -> mc60_fp:CP_Elec_10x10
- C35, C40: footprint (none) -> mc60_fp:CP_Elec_6.3x5.8
- CN1, CN2: footprint (none) -> mc60_fp:sma_smt_ra
- CN3: footprint (none) -> mc60_fp:microsd-9-suntech-ST-TF-003A
- CN4: footprint (none) -> mc60_fp:conn_microSIM_SF56S006V4BR2000
- CN5: footprint (none) -> mc60_fp:SJ2-4351-SMT
