File: kicad/mc60.sch (KiCad schematic (older format))
At the start: 98 parts, among them CN1 Conn_GPS, CN2 Conn_GNSS, CN3 SD_CARD, CN4 SIM_Card, CN5 Audio-Jack-4, J1 B_LS_N, J2 B_VRTC, J3 B_SPKP, J4 B_SPKN, J5 B_ADC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

Commit message: schematic wip
Parts:
- CN5: footprint mc60_fp:SJ2-4351-SMT -> mc60_fp:AUDIO8P-SMD-3.5-14.5X6X5MM
- D1, D4: footprint (none) -> mc60_fp:SLP1616P6
- D2, D3, D8: footprint (none) -> mc60_fp:LED_0603
- R1, R10, R11, R12, R13, R14, R15, R16, R17, R18, R19, R2, R20, R3, R4, R5, R6, R7, R8, R9: footprint Capacitors_SMD:C_0603 -> mc60_fp:R_0603
Connections:
- wire segments 468 -> 485
- no-connect marks 17 -> 16
Changed lines of the file:
@@
 U 1 1 5ACBF9E1
 P 11150 3350
-F 0 "CN4" H 11000 3225 50  0000 L CNB
-F 1 "SIM_Card" H 11000 3150 50  0000 L CNB
+F 0 "CN4" H 11050 3650 50  0000 L CNB
+F 1 "SIM_Card" H 11050 3575 50  0000 L CNB
 F 2 "mc60_fp:conn_microSIM_SF56S006V4BR2000" H 11150 3700 50  0001 C CNN
 F 3 "" H 11100 3350 50  0000 C CNN
@@
 F 0 "R1" H 9800 1100 40  0000 L CNB
 F 1 "100k" V 9750 1025 40  0000 C CNN
-F 2 "Capacitors_SMD:C_0603" V 9680 1025 30  0001 C CNN
+F 2 "mc60_fp:R_0603" V 9680 1025 30  0001 C CNN
 F 3 "" H 9750 1025 30  0000 C CNN
 	1    9750 1025
@@
 Text Label 1450 3400 0    40   ~ 8
 SD_DAT
-NoConn ~ 11650 1700
 Wire Wire Line
 	11500 1950 11500 2000
@@
 F 0 "R5" H 9025 3025 40  0000 L CNB
 F 1 "100k" V 8950 2950 40  0000 C CNN
-F 2 "Capacitors_SMD:C_0603" V 8880 2950 30  0001 C CNN
+F 2 "mc60_fp:R_0603" V 8880 2950 30  0001 C CNN
 F 3 "" H 8950 2950 30  0000 C CNN
 	1    8950 2950
@@
 F 0 "R10" V 8600 3700 40  0000 C CNB
 F 1 "22E" V 8650 3550 40  0000 C CNN
-F 2 "Capacitors_SMD:C_0603" V 8580 3550 30  0001 C CNN
+F 2 "mc60_fp:R_0603" V 8580 3550 30  0001 C CNN
 F 3 "" H 8650 3550 30  0000 C CNN
 	1    8650 3550
@@
 F 0 "R7" V 8500 3400 40  0000 C CNB
 F 1 "22E" V 8650 3250 40  0000 C CNN
-F 2 "Capacitors_SMD:C_0603" V 8580 3250 30  0001 C CNN
+F 2 "mc60_fp:R_0603" V 8580 3250 30  0001 C CNN
 F 3 "" H 8650 3250 30  0000 C CNN
 	1    8650 3250
@@
 F 0 "R6" V 8700 3300 40  0000 C CNB
 F 1 "22E" V 8650 3150 40  0000 C CNN
-F 2 "Capacitors_SMD:C_0603" V 8580 3150 30  0001 C CNN
+F 2 "mc60_fp:R_0603" V 8580 3150 30  0001 C CNN
 F 3 "" H 8650 3150 30  0000 C CNN
 	1    8650 3150
@@
 F 0 "D4" H 10525 3675 50  0000 R CNB
 F 1 "RClamp0854P.TCT" H 10425 3600 40  0000 L CNN
-F 2 "" H 10275 3875 50  0001 C CNN
+F 2 "mc60_fp:SLP1616P6" H 10275 3875 50  0001 C CNN
 F 3 "" H 10275 3875 50  0001 C CNN
 	1    10275 3875
@@
 F 0 "R8" H 12825 3600 40  0000 L CNB
 F 1 "390E" V 12750 3525 40  0000 C CNN
-F 2 "Capacitors_SMD:C_0603" V 12680 3525 30  0001 C CNN
+F 2 "mc60_fp:R_0603" V 12680 3525 30  0001 C CNN
 F 3 "" H 12750 3525 30  0000 C CNN
 	1    12750 3525
@@
 F 0 "D2" V 12725 3250 40  0000 L CNB
 F 1 "LED_NET" V 12800 3250 40  0000 L CNN
-F 2 "" H 12750 3175 60  0001 C CNN
+F 2 "mc60_fp:LED_0603" H 12750 3175 60  0001 C CNN
 F 3 "" H 12750 3175 60  0000 C CNN
 F 4 "LED SS 5MM 625NM RED DIFF" H 12750 3375 60  0001 L CNN "Field4"
@@
 F 0 "R9" H 14125 3600 40  0000 L CNB
 F 1 "270E" V 14050 3525 40  0000 C CNN
-F 2 "Capacitors_SMD:C_0603" V 13980 3525 30  0001 C CNN
+F 2 "mc60_fp:R_0603" V 13980 3525 30  0001 C CNN
 F 3 "" H 14050 3525 30  0000 C CNN
 	1    14050 3525
@@
 F 0 "D3" V 14025 3250 40  0000 L CNB
 F 1 "LED_FIX" V 14100 3250 40  0000 L CNN
-F 2 "" H 14050 3175 60  0001 C CNN
+F 2 "mc60_fp:LED_0603" H 14050 3175 60  0001 C CNN
 F 3 "" H 14050 3175 60  0000 C CNN
 F 4 "LED SS 5MM 625NM RED DIFF" H 14050 3375 60  0001 L CNN "Field4"
@@
 F 0 "R16" H 2650 8850 40  0000 L CNN
 F 1 "51k" V 2625 8700 40  0000 C CNN
-F 2 "Capacitors_SMD:C_0603" V 2555 8700 30  0001 C CNN
+F 2 "mc60_fp:R_0603" V 2555 8700 30  0001 C CNN
 F 3 "" H 2625 8700 30  0000 C CNN
 	1    2625 8700
@@
 F 0 "R17" H 3800 8850 40  0000 L CNB
 F 1 "124k" V 3775 8700 40  0000 C CNN
-F 2 "Capacitors_SMD:C_0603" V 3705 8700 30  0001 C CNN
+F 2 "mc60_fp:R_0603" V 3705 8700 30  0001 C CNN
 F 3 "" H 3775 8700 30  0000 C CNN
 	1    3775 8700
@@
 F 0 "R19" H 3800 9600 40  0000 L CNB
 F 1 "56k" V 3775 9450 40  0000 C CNN
-F 2 "Capacitors_SMD:C_0603" V 3705 9450 30  0001 C CNN
+F 2 "mc60_fp:R_0603" V 3705 9450 30  0001 C CNN
 F 3 "" H 3775 9450 30  0000 C CNN
 	1    3775 9450
@@
 F 0 "R18" H 4000 8850 40  0000 L CNB
 F 1 "390E" V 3975 8700 40  0000 C CNN
-F 2 "Capacitors_SMD:C_0603" V 3905 8700 30  0001 C CNN
+F 2 "mc60_fp:R_0603" V 3905 8700 30  0001 C CNN
 F 3 "" H 3975 8700 30  0000 C CNN
 	1    3975 8700
@@
 F 0 "R20" H 6350 9600 40  0000 L CNB
 F 1 "47k" V 6325 9450 40  0000 C CNN
-F 2 "Capacitors_SMD:C_0603" V 6255 9450 30  0001 C CNN
+F 2 "mc60_fp:R_0603" V 6255 9450 30  0001 C CNN
 F 3 "" H 6325 9450 30  0000 C CNN
 	1    6325 9450
@@
 F 0 "D8" V 3825 9475 40  0000 L CNB
 F 1 "LED_PWR" H 4050 9500 40  0000 L CNN
-F 2 "" H 3975 9450 60  0001 C CNN
+F 2 "mc60_fp:LED_0603" H 3975 9450 60  0001 C CNN
 F 3 "" H 3975 9450 60  0000 C CNN
 F 4 "LED SS 5MM 625NM RED DIFF" H 3975 9650 60  0001 L CNN "Field4"
@@
 F 0 "R11" V 2700 5250 40  0000 C CNB
 F 1 "0E" V 2750 5075 40  0000 C CNN
-F 2 "Capacitors_SMD:C_0603" V 2680 5075 30  0001 C CNN
+F 2 "mc60_fp:R_0603" V 2680 5075 30  0001 C CNN
 F 3 "" H 2750 5075 30  0000 C CNN
 	1    2750 5075
@@
 F 0 "R12" V 3550 5350 40  0000 C CNB
 F 1 "0E" V 3600 5175 40  0000 C CNN
-F 2 "Capacitors_SMD:C_0603" V 3530 5175 30  0001 C CNN
+F 2 "mc60_fp:R_0603" V 3530 5175 30  0001 C CNN
 F 3 "" H 3600 5175 30  0000 C CNN
 	1    3600 5175
@@
 F 0 "R13" V 3650 5000 40  0000 C CNB
 F 1 "0E" V 3700 5175 40  0000 C CNN
-F 2 "Capacitors_SMD:C_0603" V 3630 5175 30  0001 C CNN
+F 2 "mc60_fp:R_0603" V 3630 5175 30  0001 C CNN
 F 3 "" H 3700 5175 30  0000 C CNN
 	1    3700 5175
@@
 F 0 "R14" H 12500 6600 40  0000 L CNB
 F 1 "10k" V 12475 6450 40  0000 C CNN
-F 2 "Capacitors_SMD:C_0603" V 12405 6450 30  0001 C CNN
+F 2 "mc60_fp:R_0603" V 12405 6450 30  0001 C CNN
 F 3 "" H 12475 6450 30  0000 C CNN
 	1    12475 6450
@@
 F 0 "D1" H 10525 1775 50  0000 R CNB
 F 1 "RClamp0854P.TCT" H 10425 1700 40  0000 L CNN
-F 2 "" H 10275 1975 50  0001 C CNN
+F 2 "mc60_fp:SLP1616P6" H 10275 1975 50  0001 C CNN
 F 3 "" H 10275 1975 50  0001 C CNN
 	1    10275 1975
@@
 F 0 "R2" V 12450 1475 40  0000 C CNB
 F 1 "0E" V 12525 1475 40  0000 C CNN
-F 2 "Capacitors_SMD:C_0603" V 12455 1475 30  0001 C CNN
+F 2 "mc60_fp:R_0603" V 12455 1475 30  0001 C CNN
 F 3 "" H 12525 1475 30  0000 C CNN
 	1    12525 1475
@@
 F 0 "R3" V 13750 1475 40  0000 C CNB
 F 1 "0E" V 13825 1475 40  0000 C CNN
-F 2 "Capacitors_SMD:C_0603" V 13755 1475 30  0001 C CNN
+F 2 "mc60_fp:R_0603" V 13755 1475 30  0001 C CNN
 F 3 "" H 13825 1475 30  0000 C CNN
 	1    13825 1475
@@
 F 0 "R4" V 14925 1475 40  0000 C CNB
 F 1 "0E" V 15000 1475 40  0000 C CNN
-F 2 "Capacitors_SMD:C_0603" V 14930 1475 30  0001 C CNN
+F 2 "mc60_fp:R_0603" V 14930 1475 30  0001 C CNN
 F 3 "" H 15000 1475 30  0000 C CNN
 	1    15000 1475
@@
 F 0 "CN5" H 11475 4875 40  0000 R CNB
 F 1 "Audio-Jack-4" H 11475 4800 40  0000 R CNN
-F 2 "mc60_fp:SJ2-4351-SMT" H 11625 4825 50  0001 C CNN
+F 2 "mc60_fp:AUDIO8P-SMD-3.5-14.5X6X5MM" H 11625 4825 50  0001 C CNN
 F 3 "~" H 11625 4825 50  0001 C CNN
 F 4 "SJ-43514-SMT-TR" H 11375 4725 50  0001 C CNN "manf#"
@@
 F 0 "R15" V 10200 6650 40  0000 C CNB
 F 1 "0E" V 10275 6650 40  0000 C CNN
-F 2 "Capacitors_SMD:C_0603" V 10205 6650 30  0001 C CNN
+F 2 "mc60_fp:R_0603" V 10205 6650 30  0001 C CNN
 F 3 "" H 10275 6650 30  0000 C CNN
 	1    10275 6650
@@
 Text Label 10050 875  2    40   ~ 8
 VDD_EXT
+Wire Wire Line
+	11150 3700 11150 3750
+Wire Wire Line
+	11150 3750 11200 3750
+Wire Wire Line
+	11500 3750 11500 3700
+Wire Wire Line
+	11450 3700 11450 3750
+Connection ~ 11450 3750
+Wire Wire Line
+	11450 3750 11500 3750
+Wire Wire Line
+	11400 3700 11400 3750
+Connection ~ 11400 3750
+Wire Wire Line
+	11400 3750 11450 3750
+Wire Wire Line
+	11350 3700 11350 3750
+Connection ~ 11350 3750
+Wire Wire Line
+	11350 3750 11400 3750
+Wire Wire Line
+	11300 3700 11300 3750
+Connection ~ 11300 3750
+Wire Wire Line
+	11300 3750 11350 3750
+Wire Wire Line
+	11250 3700 11250 3750
+Connection ~ 11250 3750
+Wire Wire Line
+	11250 3750 11300 3750
+Wire Wire Line
+	11200 3700 11200 3750
+Connection ~ 11200 3750
+Wire Wire Line
+	11200 3750 11250 3750
+Wire Wire Line
+	11150 3750 11150 4175
+Wire Wire Line
+	11150 4175 10075 4175
+Connection ~ 11150 3750
+Connection ~ 10075 4175
 $EndSCHEMATC

Commit message: schematic wip
Parts:
- CN4: footprint mc60_fp:conn_microSIM_SF56S006V4BR2000 -> mc60_fp:conn_microSIM_320100004
- D5, D6: footprint (none) -> mc60_fp:D_SOD-923
- D7: footprint (none) -> mc60_fp:D_SOD-128
- H1, JP1, JP2: footprint (none) -> mc60_fp:Pin_Header_Straight_1x03
- H2, H3: footprint (none) -> mc60_fp:Pin_Header_Straight_2x04
- J1, J2, J3, J4, J5: footprint (none) -> mc60_fp:Test_Point_Plated_Hole_d2.0mm
- Q1, Q2, Q3: footprint (none) -> mc60_fp:SOT-323_SC-70
- Q4: value DTC114E -> DTC143ZUA; footprint (none) -> mc60_fp:SOT-323_SC-70
- S1: footprint (none) -> mc60_fp:SW_SPST_FSM6JSMA
- U1: footprint (none) -> mc60_fp:XCVR_MC60
- U2: footprint Package_TO_SOT_SMD:USON-20_2x4mm_P0.4mm -> mc60_fp:TSSOP-20_4.4x6.5mm_Pitch0.65mm
- U3: footprint Package_TO_SOT_SMD:TO-252-6 -> mc60_fp:TO-252-5_TabPin3
- U4, U5: footprint Package_TO_SOT_SMD:TO-252-6 -> mc60_fp:SOT-23-5
Changed lines of the file:
@@
 F 0 "U1" H 3550 3425 60  0000 C CNB
 F 1 "MC60_0" H 3550 3300 60  0000 C CNB
-F 2 "" H 3550 3050 60  0001 C BNB
+F 2 "mc60_fp:XCVR_MC60" H 3550 3050 60  0001 C BNB
 F 3 "MC60" H 3550 3550 60  0001 C BNB
 	1    3550 3300
@@
 F 0 "CN4" H 11050 3650 50  0000 L CNB
 F 1 "SIM_Card" H 11050 3575 50  0000 L CNB
-F 2 "mc60_fp:conn_microSIM_SF56S006V4BR2000" H 11150 3700 50  0001 C CNN
+F 2 "mc60_fp:conn_microSIM_320100004" H 11150 3700 50  0001 C CNN
 F 3 "" H 11100 3350 50  0000 C CNN
 	1    11150 3350
@@
 $EndComp
 Wire Wire Line
-	15550 1650 15550 1900
+	15550 1625 15550 1900
 Wire Wire Line
 	14250 1650 14250 1900
@@
 F 0 "Q1" H 12400 4150 40  0000 C CNB
 F 1 "DTC114E" H 12400 4075 40  0000 C CNN
-F 2 "" H 12150 3850 50  0001 L CNN
+F 2 "mc60_fp:SOT-323_SC-70" H 12150 3850 50  0001 L CNN
 F 3 "" H 12150 3850 50  0001 L CNN
 	1    12400 3850
@@
 F 0 "Q2" H 13700 4150 40  0000 C CNB
 F 1 "DTC114E" H 13700 4075 40  0000 C CNN
-F 2 "" H 13450 3850 50  0001 L CNN
+F 2 "mc60_fp:SOT-323_SC-70" H 13450 3850 50  0001 L CNN
 F 3 "" H 13450 3850 50  0001 L CNN
 	1    13700 3850
@@
 F 0 "Q3" H 15200 4150 40  0000 C CNB
 F 1 "DTC114E" H 15200 4075 40  0000 C CNN
-F 2 "" H 14950 3850 50  0001 L CNN
+F 2 "mc60_fp:SOT-323_SC-70" H 14950 3850 50  0001 L CNN
 F 3 "" H 14950 3850 50  0001 L CNN
 	1    15200 3850
@@
 F 0 "U3" H 3175 8875 40  0000 C CNB
 F 1 "MIC29302" H 3175 8800 40  0000 C CNN
-F 2 "Package_TO_SOT_SMD:TO-252-6" H 3175 8150 50  0001 C CIN
+F 2 "mc60_fp:TO-252-5_TabPin3" H 3175 8150 50  0001 C CIN
 F 3 "http://www.analog.com/media/en/technical-documentation/data-sheets/ADP7142.pdf" H 3175 8050 50  0001 C CNN
 	1    3175 8550
@@
 P 2375 9325
 F 0 "Q4" H 2375 9625 40  0000 C CNB
-F 1 "DTC114E" H 2375 9550 40  0000 C CNN
-F 2 "" H 2125 9325 50  0001 L CNN
+F 1 "DTC143ZUA" H 2375 9550 40  0000 C CNN
+F 2 "mc60_fp:SOT-323_SC-70" H 2125 9325 50  0001 L CNN
 F 3 "" H 2125 9325 50  0001 L CNN
 F 4 "mfr_pn" H 2375 9325 50  0001 C CNN "manf#"
@@
 F 0 "U4" H 6825 8875 40  0000 C CNB
 F 1 "LP5907-3V3" H 6825 8800 40  0000 C CNN
-F 2 "Package_TO_SOT_SMD:TO-252-6" H 6825 8150 50  0001 C CIN
+F 2 "mc60_fp:SOT-23-5" H 6825 8150 50  0001 C CIN
 F 3 "http://www.ti.com/lit/ds/symlink/lp5907-q1.pdf" H 6825 8050 50  0001 C CNN
 	1    6825 8550
@@
 F 0 "D7" V 5525 8675 40  0000 R CNB
 F 1 "PDZVTR5.1B" H 5075 8650 40  0000 L CNN
-F 2 "" H 5200 8725 60  0001 C CNN
+F 2 "mc60_fp:D_SOD-128" H 5200 8725 60  0001 C CNN
 F 3 "" H 5200 8725 60  0000 C CNN
 	1    5375 8700
@@
 F 0 "U5" H 6825 10650 40  0000 C CNB
 F 1 "LP5907-2V8" H 6825 10575 40  0000 C CNN
-F 2 "Package_TO_SOT_SMD:TO-252-6" H 6825 9925 50  0001 C CIN
+F 2 "mc60_fp:SOT-23-5" H 6825 9925 50  0001 C CIN
 F 3 "http://www.ti.com/lit/ds/symlink/lp5907-q1.pdf" H 6825 9825 50  0001 C CNN
 	1    6825 10325
@@
 F 0 "JP2" V 1275 9400 40  0000 L CNB
 F 1 "GSM_PWR_EN" V 1200 9400 40  0000 L CNN
-F 2 "" H 1200 9325 50  0001 C CNN
+F 2 "mc60_fp:Pin_Header_Straight_1x03" H 1200 9325 50  0001 C CNN
 F 3 "~" H 1200 9325 50  0001 C CNN
 F 4 "mfr_pn" H 1200 9325 50  0001 C CNN "manf#"
@@
 F 0 "U2" H 13200 5175 40  0000 L CNB
 F 1 "TXB0108PWR" H 13200 5100 40  0000 L CNN
-F 2 "Package_TO_SOT_SMD:USON-20_2x4mm_P0.4mm" H 13325 6275 50  0001 L CNN
+F 2 "mc60_fp:TSSOP-20_4.4x6.5mm_Pitch0.65mm" H 13325 6275 50  0001 L CNN
 F 3 "http://www.ti.com/lit/ds/symlink/txb0108.pdf" H 12975 5725 50  0001 C CNN
 	1    12975 5825
@@
 F 0 "JP1" H 13500 5050 50  0000 C CNB
 F 1 "3V3_EXT<>5V" H 13500 4950 40  0000 C CNN
-F 2 "" H 13500 4825 50  0001 C CNN
+F 2 "mc60_fp:Pin_Header_Straight_1x03" H 13500 4825 50  0001 C CNN
 F 3 "~" H 13500 4825 50  0001 C CNN
 F 4 "mfr_pn" H 13500 4825 50  0001 C CNN "manf#"
@@
 F 0 "D6" V 9850 6125 40  0000 L CNB
 F 1 "ESD9B5.0ST5G" V 10100 6075 40  0000 L CNN
-F 2 "" H 9950 6050 50  0001 C CNN
+F 2 "mc60_fp:D_SOD-923" H 9950 6050 50  0001 C CNN
 F 3 "https://en.wikipedia.org/wiki/Transient-voltage-suppression_diode" H 9950 6050 50  0001 C CNN
 	1    9950 6050
@@
 F 0 "D5" V 9850 5000 40  0000 L CNB
 F 1 "ESD9B5.0ST5G" V 10100 4950 40  0000 L CNN
-F 2 "" H 9950 4925 50  0001 C CNN
+F 2 "mc60_fp:D_SOD-923" H 9950 4925 50  0001 C CNN
 F 3 "https://en.wikipedia.org/wiki/Transient-voltage-suppression_diode" H 9950 4925 50  0001 C CNN
 	1    9950 4925
@@
 F 0 "J3" H 1650 2800 40  0000 L CNN
 F 1 "B_SPKP" H 1375 2800 40  0000 L CNN
-F 2 "" H 1300 2800 50  0001 C CNN
+F 2 "mc60_fp:Test_Point_Plated_Hole_d2.0mm" H 1300 2800 50  0001 C CNN
 F 3 "" H 1300 2800 50  0001 C CNN
 	1    1300 2800
@@
 F 0 "J4" H 1650 2900 40  0000 L CNN
 F 1 "B_SPKN" H 1375 2900 40  0000 L CNN
-F 2 "" H 1300 2900 50  0001 C CNN
+F 2 "mc60_fp:Test_Point_Plated_Hole_d2.0mm" H 1300 2900 50  0001 C CNN
 F 3 "" H 1300 2900 50  0001 C CNN
 	1    1300 2900
@@
 F 0 "J5" H 1650 3100 40  0000 L CNN
 F 1 "B_ADC" H 1375 3100 40  0000 L CNN
-F 2 "" H 1300 3100 50  0001 C CNN
+F 2 "mc60_fp:Test_Point_Plated_Hole_d2.0mm" H 1300 3100 50  0001 C CNN
 F 3 "" H 1300 3100 50  0001 C CNN
 	1    1300 3100
@@
 F 0 "J1" H 3450 1050 40  0000 L CNN
 F 1 "B_LS_N" H 3175 1050 40  0000 L CNN
-F 2 "" H 3100 1050 50  0001 C CNN
+F 2 "mc60_fp:Test_Point_Plated_Hole_d2.0mm" H 3100 1050 50  0001 C CNN
 F 3 "" H 3100 1050 50  0001 C CNN
 	1    3100 1050
@@
 F 0 "J2" H 3550 1050 40  0000 L CNN
 F 1 "B_VRTC" H 3275 1050 40  0000 L CNN
-F 2 "" H 3200 1050 50  0001 C CNN
+F 2 "mc60_fp:Test_Point_Plated_Hole_d2.0mm" H 3200 1050 50  0001 C CNN
 F 3 "" H 3200 1050 50  0001 C CNN
 	1    3200 1050
@@
 F 0 "S1" V 14700 3900 40  0000 R CNB
 F 1 "SW-ON" V 14575 3900 40  0000 R CNN
-F 2 "" H 14700 3650 60  0001 C CNN
+F 2 "mc60_fp:SW_SPST_FSM6JSMA" H 14700 3650 60  0001 C CNN
 F 3 "" H 14700 3650 60  0000 C CNN
 F 4 "mfr_pn" H 14700 3650 50  0001 C CNN "manf#"
@@
 F 0 "H1" H 15475 5300 40  0000 L CNB
 F 1 "UART_DBG" H 15475 5225 40  0000 L CNN
-F 2 "" H 15375 5250 50  0001 C CNN
+F 2 "mc60_fp:Pin_Header_Straight_1x03" H 15375 5250 50  0001 C CNN
 F 3 "~" H 15375 5250 50  0001 C CNN
 	1    15375 5250
@@
 F 0 "H3" H 15475 5950 40  0000 L CNB
 F 1 "CONTROL" H 15475 5875 40  0000 L CNN
-F 2 "" H 15375 5900 50  0001 C CNN
+F 2 "mc60_fp:Pin_Header_Straight_2x04" H 15375 5900 50  0001 C CNN
 F 3 "" H 15375 5900 50  0000 C CNN
 	1    15375 5900
@@
 F 0 "H2" H 14075 5925 40  0000 L CNB
 F 1 "UART" H 14075 5850 40  0000 L CNN
-F 2 "" H 13975 5875 50  0001 C CNN
+F 2 "mc60_fp:Pin_Header_Straight_2x04" H 13975 5875 50  0001 C CNN
 F 3 "" H 13975 5875 50  0000 C CNN
 	1    13975 5875

Commit message: schematic wip
Changed lines of the file:
@@
 	10650 3150 10225 3150
 Wire Wire Line
-	10650 3350 9725 3350
-Wire Wire Line
 	9725 3350 9725 4175
 Wire Wire Line
@@
 	8950 3100 8950 3550
 Wire Wire Line
-	8950 3550 10425 3550
+	8950 3550 10325 3550
 $Comp
 L mc60_library:R R10
@@
 Connection ~ 9150 3250
 Wire Wire Line
-	9150 3250 10325 3250
-Wire Wire Line
 	8950 3675 8950 3550
 Wire Wire Line
@@
 $EndComp
 Wire Wire Line
-	10425 3625 10425 3550
-Connection ~ 10425 3550
-Wire Wire Line
-	10425 3550 10650 3550
-Wire Wire Line
-	10325 3625 10325 3250
-Connection ~ 10325 3250
-Wire Wire Line
-	10325 3250 10650 3250
-Wire Wire Line
 	10225 3625 10225 3150
 Connection ~ 10225 3150
@@
 Connection ~ 11150 3750
 Connection ~ 10075 4175
+Wire Wire Line
+	9150 3250 10425 3250
+Wire Wire Line
+	10325 3625 10325 3550
+Connection ~ 10325 3550
+Wire Wire Line
+	10325 3550 10650 3550
+Wire Wire Line
+	9725 3350 10650 3350
+Wire Wire Line
+	10425 3625 10425 3250
+Connection ~ 10425 3250
+Wire Wire Line
+	10425 3250 10650 3250
 $EndSCHEMATC

Commit message: layout WIP
Parts:
- C10, C11, C13, C14, C16, C17, C18, C19, C20, C21, C22, C23, C24, C25, C28, C32, C33, C34, C36, C39, C41, C44, C8, C9: footprint mc60_fp:C_0603 -> mc60_fp:C_0402_NoSilk
- C35, C40: footprint mc60_fp:CP_Elec_6.3x5.8 -> mc60_fp:CP_Elec_8x10.5
- CN1, CN2: footprint mc60_fp:sma_smt_ra -> mc60_fp:Molex_Microcoaxial_RF
- J1, J2, J3, J4, J5: footprint mc60_fp:Test_Point_Plated_Hole_d2.0mm -> mc60_fp:Test_Point_Pad_2.0x2.0mm
- R11, R12, R13, R15, R2, R3, R4: footprint mc60_fp:R_0603 -> mc60_fp:R_0402_NoSilk
- S1: footprint mc60_fp:SW_SPST_FSM6JSMA -> mc60_fp:SW_SPST_DTSM

Commit message: layout wip
Parts:
- added CN6: 5V_IN, mc60_fp:conn_screw_2.54mm_2pol, symbol mc60_library:Conn_01x02
Connections:
- wire segments 485 -> 491
Changed lines of the file:
@@
 U 1 1 5AFB7208
 P 1200 9325
-F 0 "JP2" V 1275 9400 40  0000 L CNB
-F 1 "GSM_PWR_EN" V 1200 9400 40  0000 L CNN
+F 0 "JP2" V 1325 9350 40  0000 L CNB
+F 1 "GSM_PWR_EN" H 1100 9375 40  0000 R CNN
 F 2 "mc60_fp:Pin_Header_Straight_1x03" H 1200 9325 50  0001 C CNN
 F 3 "~" H 1200 9325 50  0001 C CNN
@@
 Wire Wire Line
 	10425 3250 10650 3250
+$Comp
+L mc60_library:Conn_01x02 CN6
+U 1 1 5AE1C71C
+P 700 9275
+F 0 "CN6" H 600 9500 40  0000 C CNB
+F 1 "5V_IN" H 600 9400 40  0000 C CNN
+F 2 "mc60_fp:conn_screw_2.54mm_2pol" H 700 9275 50  0001 C CNN
+F 3 "" H 700 9275 50  0001 C CNN
+	1    700  9275
+	-1   0    0    -1
+$EndComp
+Wire Wire Line
+	900  9275 1000 9275
+Wire Wire Line
+	1000 9275 1000 8450
+Wire Wire Line
+	1000 8450 1200 8450
+Connection ~ 1200 8450
+Wire Wire Line
+	900  9375 1000 9375
+Wire Wire Line
+	1000 9375 1000 9775
+Wire Wire Line
+	1000 9775 1200 9775
 $EndSCHEMATC

Commit message: layout WIP
Connections:
- net labels added: SIMCLK, SIMDAT, SIMRST
Changed lines of the file:
@@
 Wire Wire Line
 	1000 9775 1200 9775
+Text Label 9800 3150 0    40   ~ 8
+SIMRST
+Text Label 9800 3250 0    40   ~ 8
+SIMCLK
+Text Label 9800 3550 0    40   ~ 8
+SIMDAT
 $EndSCHEMATC

Commit message: layout wip
Parts:
- H3: footprint mc60_fp:Pin_Header_Straight_2x04 -> mc60_fp:Pin_Header_Straight_2x04_Pitch1.27mm
- JP1, JP2: footprint mc60_fp:Pin_Header_Straight_1x03 -> mc60_fp:Pin_Header_Straight_1x03_Pitch1.27mm
Changed lines of the file:
@@
 F 0 "JP2" V 1325 9350 40  0000 L CNB
 F 1 "GSM_PWR_EN" H 1100 9375 40  0000 R CNN
-F 2 "mc60_fp:Pin_Header_Straight_1x03" H 1200 9325 50  0001 C CNN
+F 2 "mc60_fp:Pin_Header_Straight_1x03_Pitch1.27mm" H 1200 9325 50  0001 C CNN
 F 3 "~" H 1200 9325 50  0001 C CNN
 F 4 "mfr_pn" H 1200 9325 50  0001 C CNN "manf#"
@@
 F 0 "JP1" H 13500 5050 50  0000 C CNB
 F 1 "3V3_EXT<>5V" H 13500 4950 40  0000 C CNN
-F 2 "mc60_fp:Pin_Header_Straight_1x03" H 13500 4825 50  0001 C CNN
+F 2 "mc60_fp:Pin_Header_Straight_1x03_Pitch1.27mm" H 13500 4825 50  0001 C CNN
 F 3 "~" H 13500 4825 50  0001 C CNN
 F 4 "mfr_pn" H 13500 4825 50  0001 C CNN "manf#"
@@
 	1    0    0    -1
 $EndComp
-Text Label 14650 5950 0    40   ~ 8
+Text Label 14650 6250 0    40   ~ 8
 GND
 Text Label 14650 6050 0    40   ~ 8
 GND
-Text Label 14650 6250 0    40   ~ 8
+Text Label 14650 5950 0    40   ~ 8
 5V
 $Comp
@@
 F 0 "H3" H 15475 5950 40  0000 L CNB
 F 1 "CONTROL" H 15475 5875 40  0000 L CNN
-F 2 "mc60_fp:Pin_Header_Straight_2x04" H 15375 5900 50  0001 C CNN
+F 2 "mc60_fp:Pin_Header_Straight_2x04_Pitch1.27mm" H 15375 5900 50  0001 C CNN
 F 3 "" H 15375 5900 50  0000 C CNN
 	1    15375 5900
@@
 Text Label 9175 6725 0    40   ~ 8
 GND_REF
-Wire Notes Line
-	14600 6150 14550 6150
-Wire Notes Line
-	14550 6150 14525 6125
-Wire Notes Line
-	14525 6125 14525 6075
-Wire Notes Line
-	14525 6075 14550 6050
-Wire Notes Line
-	14550 6050 14600 6050
-Wire Notes Line
-	14550 6150 14525 6175
-Wire Notes Line
-	14525 6175 14525 6225
-Wire Notes Line
-	14525 6225 14550 6250
-Wire Notes Line
-	14550 6250 14600 6250
-Wire Notes Line
-	14600 5850 14550 5850
-Wire Notes Line
-	14550 5850 14525 5825
-Wire Notes Line
-	14525 5825 14525 5775
-Wire Notes Line
-	14525 5775 14550 5750
-Wire Notes Line
-	14550 5750 14600 5750
-Wire Notes Line
-	14550 5850 14525 5875
-Wire Notes Line
-	14525 5875 14525 5925
-Wire Notes Line
-	14525 5925 14550 5950
-Wire Notes Line
-	14550 5950 14600 5950
 Text Label 12325 1900 0    40   ~ 8
 GND
@@
 Text Label 9800 3550 0    40   ~ 8
 SIMDAT
+Wire Notes Line
+	14625 5850 14450 5850
+Wire Notes Line
+	14450 5750 14625 5750
+Wire Notes Line
+	14450 6050 14625 6050
+Wire Notes Line
+	14450 5750 14450 6050
+Wire Notes Line
+	14625 6150 14525 6150
+Wire Notes Line
+	14525 5950 14625 5950
+Wire Notes Line
+	14525 6250 14625 6250
+Wire Notes Line
+	14525 5950 14525 6250
 $EndSCHEMATC
