File: kicad/mc60.sch (KiCad schematic (older format))
At the start: 107 parts, among them CN1 Conn_GPS, CN2 Conn_GNSS, CN3 SD_CARD, CN4 SIM_Card, CN5 Audio-Jack-4, CN6 5V_IN, J1 B_LS_N, J2 B_VRTC, J3 B_SPKP, J4 B_SPKN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

Commit message: layout WIP
Parts:
- H4: value ON_OFF -> ON<>OFF
Other:
- note added: "Power control\nPush S1 for ON, Push S1 for OFF\nOR via external "RST" signal on H4"
- note removed: "Power control\nPush S1 for ON, Push S1 for OFF\nOR via external "RST" signal"
Changed lines of the file:
@@
 Text Notes 14400 4575 0    50   Italic 10
 HEADERS
-Text Notes 1875 8250 0    50   Italic 10
+Text Notes 625  8325 0    50   Italic 10
 5V/3A (2A min)
 Text Notes 4525 8250 0    50   Italic 10
@@
 Text Notes 11875 6850 0    40   ~ 0
 UART output voltage can be either\n5V (derived from main input) or\n3V3 (derived from external input)
-Text Notes 600  10075 0    40   ~ 0
+Text Notes 600  10125 0    40   ~ 0
 JP2 > 5V = OFF (VReg U3 is disabled).\nJP2 > GND = ON (VReg U3 is enabled).\n
-Text Notes 14750 2875 0    40   ~ 0
-Power control\nPush S1 for ON, Push S1 for OFF\nOR via external "RST" signal
+Text Notes 14725 2875 0    40   ~ 0
+Power control\nPush S1 for ON, Push S1 for OFF\nOR via external "RST" signal on H4
 Text Notes 13250 2850 0    40   ~ 0
 LED flashes at 1pps\nafter GPS fix
@@
 P 15375 6050
 F 0 "H4" H 15455 6085 40  0000 L CNB
-F 1 "ON_OFF" H 15455 6010 40  0000 L CNN
+F 1 "ON<>OFF" H 15455 6010 40  0000 L CNN
 F 2 "mc60_fp:Pin_Header_Straight_1x03" H 15375 6050 50  0001 C CNN
 F 3 "~" H 15375 6050 50  0001 C CNN

Commit message: layout WIP
Other:
- note added: "CTIA STYLE\nTRRS\nCONNECTION"
- note removed: "CITA STYLE\nTRRS\nCONNECTION"
Changed lines of the file:
@@
 $EndBitmap
 Text Notes 11025 5825 0    50   Italic 10
-CITA STYLE\nTRRS\nCONNECTION
+CTIA STYLE\nTRRS\nCONNECTION
 Text Label 10725 4825 0    40   ~ 8
 RIGHT

Commit message: UART header update, added freeite bead on Loudspeaker, added Cap for Switch
Parts:
- added C45: 33pF, mc60_fp:C_0402_NoSilk, symbol mc60_library:C_NP
- added L1: 0E, mc60_fp:R_0402_NoSilk, symbol mc60_library:IND_FERRITE_BEAD
- H1: footprint mc60_fp:Pin_Header_Straight_1x03 -> mc60_fp:Pin_Header_Straight_1x04; symbol mc60_library:Conn_01x03 -> mc60_library:Conn_01x04; manf# (none) -> mfr_pn
Connections:
- net labels added: L_SP
- wire segments 489 -> 493
Other:
- note added: "*USE FERRITE BEAD\nIF NECESSARY*"
Changed lines of the file:
@@
 Wire Wire Line
 	9750 5150 9950 5150
-Wire Wire Line
-	9550 4725 7875 4725
-Connection ~ 9550 4725
 Text Label 7875 4725 0    40   ~ 8
 LOUD_SPKP
@@
 5V
 $Comp
-L mc60_library:Conn_01x03 H1
+L mc60_library:Conn_01x04 H1
 U 1 1 5CF7EB7F
-P 15375 5250
-F 0 "H1" H 15475 5300 40  0000 L CNB
-F 1 "UART_DBG" H 15475 5225 40  0000 L CNN
-F 2 "mc60_fp:Pin_Header_Straight_1x03" H 15375 5250 50  0001 C CNN
-F 3 "~" H 15375 5250 50  0001 C CNN
-	1    15375 5250
+P 15375 5150
+F 0 "H1" H 15475 5200 40  0000 L CNB
+F 1 "UART_DBG" H 15475 5125 40  0000 L CNN
+F 2 "mc60_fp:Pin_Header_Straight_1x04" H 15375 5150 50  0001 C CNN
+F 3 "~" H 15375 5150 50  0001 C CNN
+F 4 "mfr_pn" H 15375 5150 50  0001 C CNN "manf#"
+	1    15375 5150
 	1    0    0    -1
 $EndComp
@@
 	1    0    0    -1
 $EndComp
+Wire Wire Line
+	15175 5050 14650 5050
+Text Label 14650 5050 0    40   ~ 8
+VDD_EXT
+$Comp
+L mc60_library:IND_FERRITE_BEAD L1
+U 1 1 5B003379
+P 9075 4725
+F 0 "L1" H 9075 4850 40  0000 C CNN
+F 1 "0E" H 9075 4625 40  0000 C CNN
+F 2 "mc60_fp:R_0402_NoSilk" H 9075 4725 60  0001 C CNN
+F 3 "" H 9040 4815 60  0000 C CNN
+F 4 "mfr_pn" H 9075 4725 50  0001 C CNN "manf#"
+	1    9075 4725
+	1    0    0    -1
+$EndComp
+Wire Wire Line
+	9550 4725 9275 4725
+Connection ~ 9550 4725
+Wire Wire Line
+	8875 4725 7875 4725
+Text Label 10000 4725 0    40   ~ 8
+L_SP
+Text Notes 8875 4975 0    30   ~ 6
+*USE FERRITE BEAD\nIF NECESSARY*
+$Comp
+L mc60_library:C_NP C45
+U 1 1 5B0C20C4
+P 14750 4025
+F 0 "C45" H 14900 3925 40  0000 R CNB
+F 1 "33pF" H 14925 4125 40  0000 R CNN
+F 2 "mc60_fp:C_0402_NoSilk" H 14750 4025 60  0001 C CNN
+F 3 "" H 14750 4025 60  0000 C CNN
+	1    14750 4025
+	-1   0    0    1
+$EndComp
+Wire Wire Line
+	14750 3875 14750 3850
+Wire Wire Line
+	14750 4175 14750 4200
+Connection ~ 14750 4200
 $EndSCHEMATC

Commit message: board layout WIP
Parts:
- G2: footprint mc60_fp:KiCad-Logo2_6mm_SilkScreen -> mc60_fp:KiCad-Logo3_6mm_SilkScreen
- G3: footprint mc60_fp:Logo-WL3 -> mc60_fp:logo_wyo3
- SC1, SC2, SC3, SC4: symbol mc60_library:SCREW -> mc60_library:Conn_01x01; manf# (none) -> Value
Changed lines of the file:
@@
 	14650 5550 15175 5550
 $Comp
-L mc60_library:SCREW SC1
+L mc60_library:Conn_01x01 SC1
 U 1 1 5B06DB34
 P 12000 9000
@@
 F 2 "mc60_fp:mtg_hole_3mm_vias_2" H 12000 9000 60  0001 C CNN
 F 3 "" H 12000 9000 60  0000 C CNN
+F 4 "Value" H 12000 9000 50  0001 C CNN "manf#"
 	1    12000 9000
-	1    0    0    -1
+	0    -1   -1   0
 $EndComp
 $Comp
-L mc60_library:SCREW SC2
+L mc60_library:Conn_01x01 SC2
 U 1 1 5B06DFE3
 P 12500 9000
@@
 F 2 "mc60_fp:mtg_hole_3mm_vias_2" H 12500 9000 60  0001 C CNN
 F 3 "" H 12500 9000 60  0000 C CNN
+F 4 "Value" H 12500 9000 50  0001 C CNN "manf#"
 	1    12500 9000
-	1    0    0    -1
+	0    -1   -1   0
 $EndComp
 $Comp
-L mc60_library:SCREW SC3
+L mc60_library:Conn_01x01 SC3
 U 1 1 5B06E0FB
 P 13000 9000
@@
 F 2 "mc60_fp:mtg_hole_3mm_vias_2" H 13000 9000 60  0001 C CNN
 F 3 "" H 13000 9000 60  0000 C CNN
+F 4 "Value" H 13000 9000 50  0001 C CNN "manf#"
 	1    13000 9000
-	1    0    0    -1
+	0    -1   -1   0
 $EndComp
 $Comp
-L mc60_library:SCREW SC4
+L mc60_library:Conn_01x01 SC4
 U 1 1 5B06E1FD
 P 13500 9000
@@
 F 2 "mc60_fp:mtg_hole_3mm_vias_2" H 13500 9000 60  0001 C CNN
 F 3 "" H 13500 9000 60  0000 C CNN
+F 4 "Value" H 13500 9000 50  0001 C CNN "manf#"
 	1    13500 9000
-	1    0    0    -1
+	0    -1   -1   0
 $EndComp
 Text Notes 12525 9225 0    40   ~ 0
@@
 F 0 "G2" H 15225 9982 60  0001 C CNN
 F 1 "KiCad" H 15225 10518 60  0001 C CNN
-F 2 "mc60_fp:KiCad-Logo2_6mm_SilkScreen" H 15225 10250 60  0001 C CNN
+F 2 "mc60_fp:KiCad-Logo3_6mm_SilkScreen" H 15225 10250 60  0001 C CNN
 F 3 "" H 15225 10250 60  0001 C CNN
 F 4 "Value" H 15225 10250 50  0001 C CNN "manf#"
@@
 F 0 "G3" H 12025 10164 60  0001 C CNN
 F 1 "LOGO_WL" H 12025 10436 60  0001 C CNN
-F 2 "mc60_fp:Logo-WL3" H 12025 10300 60  0001 C CNN
+F 2 "mc60_fp:logo_wyo3" H 12025 10300 60  0001 C CNN
 F 3 "" H 12025 10300 60  0001 C CNN
 F 4 "Value" H 12025 10300 50  0001 C CNN "manf#"
@@
 	14750 4175 14750 4200
 Connection ~ 14750 4200
+$Comp
+L power:GND #PWR0101
+U 1 1 5B33A221
+P 12000 9150
+F 0 "#PWR0101" H 12000 9150 30  0001 C CNN
+F 1 "GND" H 12000 9075 30  0001 C CNN
+F 2 "" H 12000 9150 60  0000 C CNN
+F 3 "" H 12000 9150 60  0000 C CNN
+F 4 "mfr_pn" H 12000 9150 50  0001 C CNN "manf#"
+	1    12000 9150
+	1    0    0    -1
+$EndComp
+$Comp
+L power:GND #PWR0102
+U 1 1 5B33A726
+P 12500 9150
+F 0 "#PWR0102" H 12500 9150 30  0001 C CNN
+F 1 "GND" H 12500 9075 30  0001 C CNN
+F 2 "" H 12500 9150 60  0000 C CNN
+F 3 "" H 12500 9150 60  0000 C CNN
+F 4 "mfr_pn" H 12500 9150 50  0001 C CNN "manf#"
+	1    12500 9150
+	1    0    0    -1
+$EndComp
+$Comp
+L power:GND #PWR0103
+U 1 1 5B33A807
+P 13000 9150
+F 0 "#PWR0103" H 13000 9150 30  0001 C CNN
+F 1 "GND" H 13000 9075 30  0001 C CNN
+F 2 "" H 13000 9150 60  0000 C CNN
+F 3 "" H 13000 9150 60  0000 C CNN
+F 4 "mfr_pn" H 13000 9150 50  0001 C CNN "manf#"
+	1    13000 9150
+	1    0    0    -1
+$EndComp
+$Comp
+L power:GND #PWR0104
+U 1 1 5B33A9BC
+P 13500 9150
+F 0 "#PWR0104" H 13500 9150 30  0001 C CNN
+F 1 "GND" H 13500 9075 30  0001 C CNN
+F 2 "" H 13500 9150 60  0000 C CNN
+F 3 "" H 13500 9150 60  0000 C CNN
+F 4 "mfr_pn" H 13500 9150 50  0001 C CNN "manf#"
+	1    13500 9150
+	1    0    0    -1
+$EndComp
 $EndSCHEMATC
