File: kicad/mc60.kicad_pcb (KiCad board)
At the start: 2 copper layers, 98 parts, among them CN1 Conn_GPS, CN2 Conn_GNSS, CN3 SD_CARD, CN4 SIM_Card, CN5 Audio-Jack-4, J1 B_LS_N, J2 B_VRTC, J3 B_SPKP, J4 B_SPKN, J5 B_ADC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

Commit message: schematic wip
Parts:
- C10, C11, C9, D4: moved to B.Cu
- moved C12 130.9 mm to (197.6, 88.8)
- moved C13 130.9 mm to (196.7, 99.2)
- moved C14 130.9 mm to (176.2, 120.6)
- moved C16 130.9 mm to (209.6, 82.1)
- moved C17 130.9 mm to (162.1, 128.5)
- moved C18 130.9 mm to (172.0, 125.1)
- moved C20 130.9 mm to (202.8, 93.9)
- moved C23 130.9 mm to (214.3, 80.4)
- moved C25 130.9 mm to (190.3, 108.9)
- moved D2 130.9 mm to (156.2, 130.2)
- moved D3 130.9 mm to (120.7, 125.3)
- moved D5 130.9 mm to (112.8, 133.3)
- moved D6 130.9 mm to (159.8, 124.5)
- moved H1 130.9 mm to (140.8, 111.2)
- moved H2 130.9 mm to (147.7, 78.7)
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Connections:
- D4 pad 1: Net-(C8-Pad2) -> Net-(C9-Pad2)
- D4 pad 2: Net-(C9-Pad2) -> Net-(C8-Pad2)
- U3 pad 1: VDD -> Net-(Q4-Pad3)
- U3 pad 2: GND -> VDD
- U3 pad 3: Net-(Q4-Pad3) -> GND
- U3 pad 4: Net-(R17-Pad2) -> VBAT
- U3 pad 5: VBAT -> Net-(R17-Pad2)

Commit message: layout WIP
Parts:
- C10, C11, C13, C14, C16, C17, C18, C19, C20, C21, C22, C23, C24, C25, C28, C32, C33, C34, C36, C39, C41, C44, C8, C9: footprint mc60_fp:C_0603 -> mc60_fp:C_0402_NoSilk
- C35, C40: footprint mc60_fp:CP_Elec_6.3x5.8 -> mc60_fp:CP_Elec_8x10.5
- CN1, CN2: footprint mc60_fp:sma_smt_ra -> mc60_fp:Molex_Microcoaxial_RF
- D1: moved to B.Cu
- J1, J2, J3, J4, J5: footprint mc60_fp:Test_Point_Plated_Hole_d2.0mm -> mc60_fp:Test_Point_Pad_2.0x2.0mm; moved to B.Cu
- R11, R12, R13, R15, R2, R3, R4: footprint mc60_fp:R_0603 -> mc60_fp:R_0402_NoSilk
- S1: footprint mc60_fp:SW_SPST_FSM6JSMA -> mc60_fp:SW_SPST_DTSM
- moved C21 129.2 mm to (90.0, 93.5), turned to 90 degrees
- moved C23 127.4 mm to (87.0, 84.6), turned to 180 degrees
- moved Q3 124.8 mm to (76.6, 104.4)
- moved J3 121.5 mm to (88.0, 92.5)
- moved C24 120.2 mm to (87.0, 94.8), turned to 90 degrees
- moved R9 117.0 mm to (85.5, 111.5)
- moved C20 113.8 mm to (89.0, 93.5), turned to 90 degrees
- moved C12 113.3 mm to (84.8, 78.2), turned to 180 degrees
- moved C13 108.2 mm to (89.6, 83.6), turned to 180 degrees
- moved JP2 107.4 mm to (123.8, 69.8), turned to 180 degrees
- moved J5 105.0 mm to (88.0, 98.0)
- moved C15 104.0 mm to (84.8, 80.2), turned to 180 degrees
- moved C25 103.3 mm to (88.0, 94.8), turned to 90 degrees
- moved C22 100.9 mm to (87.0, 83.6), turned to 180 degrees
- moved Q2 100.2 mm to (88.5, 111.5), turned to 180 degrees
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Connections:
- CN3 pad 1: (no net) -> Net-(CN3-Pad1)
- CN3 pad 2: (no net) -> Net-(CN3-Pad2)
- CN3 pad 8: (no net) -> Net-(CN3-Pad8)
- CN4 pad P6: (no net) -> Net-(CN4-PadP6)
- D1 pad 4: (no net) -> Net-(D1-Pad4)
- D1 pad 5: (no net) -> Net-(D1-Pad5)
- D4 pad 4: (no net) -> Net-(D4-Pad4)
- D4 pad 5: (no net) -> Net-(D4-Pad5)
- U1 pad 10: (no net) -> Net-(U1-Pad10)
- U1 pad 11: (no net) -> Net-(U1-Pad11)
- U1 pad 12: (no net) -> Net-(U1-Pad12)
- U1 pad 13: (no net) -> Net-(U1-Pad13)
- U1 pad 46: (no net) -> Net-(U1-Pad46)
- U1 pad 55: (no net) -> Net-(U1-Pad55)
- U1 pad 56: (no net) -> Net-(U1-Pad56)
- U1 pad 57: (no net) -> Net-(U1-Pad57)
- U1 pad 58: (no net) -> Net-(U1-Pad58)
- U1 pad 59: (no net) -> Net-(U1-Pad59)
- U1 pad 60: (no net) -> Net-(U1-Pad60)
- U1 pad 61: (no net) -> Net-(U1-Pad61)
- U1 pad 62: (no net) -> Net-(U1-Pad62)
- U1 pad 63: (no net) -> Net-(U1-Pad63)
- U1 pad 64: (no net) -> Net-(U1-Pad64)
- U1 pad 65: (no net) -> Net-(U1-Pad65)
- U1 pad 66: (no net) -> Net-(U1-Pad66)
- U1 pad 67: (no net) -> Net-(U1-Pad67)
- U1 pad 68: (no net) -> Net-(U1-Pad68)
Other:
- board outline added: 60 x 70 mm

Commit message: layout wip
Parts:
- added CN6: 5V_IN, mc60_fp:conn_screw_2.54mm_2pol, F.Cu at (77.8, 69.0)
- C10, C11, C9: moved to F.Cu
- moved C11 3.26 mm to (87.0, 125.0)
- moved U2 1.75 mm to (114.5, 102.0)
- moved R14 1.70 mm to (114.5, 97.7)
- moved C16 1.50 mm to (113.2, 106.0)
- moved C17 1.50 mm to (115.8, 106.0)
- moved C8 1.12 mm to (89.5, 123.5), turned to 180 degrees
- moved R5 0.70 mm to (87.0, 123.5)
- moved Q1 0.60 mm to (116.3, 88.1)
- moved R8 0.38 mm to (118.9, 88.1)
- moved C5 0.25 mm to (85.8, 106.2)
- moved R3 0.25 mm to (87.5, 107.0)
- moved D2 0.21 mm to (120.6, 88.1)
- moved C10 0.10 mm to (89.5, 121.2)
- moved C4 0.10 mm to (89.1, 106.2)
- moved C9 0.10 mm to (89.5, 118.0)
Connections:
- CN3 pad 1: Net-(CN3-Pad1) -> (no net)
- CN3 pad 2: Net-(CN3-Pad2) -> (no net)
- CN3 pad 8: Net-(CN3-Pad8) -> (no net)
- CN4 pad P6: Net-(CN4-PadP6) -> (no net)
- D1 pad 4: Net-(D1-Pad4) -> (no net)
- D1 pad 5: Net-(D1-Pad5) -> (no net)
- D4 pad 4: Net-(D4-Pad4) -> (no net)
- D4 pad 5: Net-(D4-Pad5) -> (no net)
- U1 pad 10: Net-(U1-Pad10) -> (no net)
- U1 pad 11: Net-(U1-Pad11) -> (no net)
- U1 pad 12: Net-(U1-Pad12) -> (no net)
- U1 pad 13: Net-(U1-Pad13) -> (no net)
- U1 pad 46: Net-(U1-Pad46) -> (no net)
- U1 pad 55: Net-(U1-Pad55) -> (no net)
- U1 pad 56: Net-(U1-Pad56) -> (no net)
- U1 pad 57: Net-(U1-Pad57) -> (no net)
- U1 pad 58: Net-(U1-Pad58) -> (no net)
- U1 pad 59: Net-(U1-Pad59) -> (no net)
- U1 pad 60: Net-(U1-Pad60) -> (no net)
- U1 pad 61: Net-(U1-Pad61) -> (no net)
- U1 pad 62: Net-(U1-Pad62) -> (no net)
- U1 pad 63: Net-(U1-Pad63) -> (no net)
- U1 pad 64: Net-(U1-Pad64) -> (no net)
- U1 pad 65: Net-(U1-Pad65) -> (no net)
- U1 pad 66: Net-(U1-Pad66) -> (no net)
- U1 pad 67: Net-(U1-Pad67) -> (no net)
- U1 pad 68: Net-(U1-Pad68) -> (no net)
Routing:
- net GND: track 0.00 -> 27.5 mm
- net /ANT_GPS: track 0.00 -> 4.39 mm
- net Net-(C3-Pad2): track 0.00 -> 2.81 mm
- added copper zone on F.Cu, net GND
Other:
- net class 0.5mm added: clearance 0.2, trace_width 0.5, via_dia 0.8, via_drill 0.4
- net class 0.70mm added: clearance 0.2, trace_width 0.7, via_dia 0.8, via_drill 0.4
- net class 1.00mm added: clearance 0.2, trace_width 1, via_dia 0.8, via_drill 0.4
- net class 1.50mm added: clearance 0.2, trace_width 1.5, via_dia 0.8, via_drill 0.4
- net class 2.00mm added: clearance 0.2, trace_width 2, via_dia 0.8, via_drill 0.4
- net class 2.50mm added: clearance 0.2, trace_width 2.5, via_dia 0.8, via_drill 0.4

Commit message: layout WIP
Parts:
- D4: moved to F.Cu
- moved D4 10.6 mm to (88.2, 128.2), turned to 180 degrees
- moved C8 5.92 mm to (88.1, 117.8)
- moved C9 3.00 mm to (88.1, 115.3)
- moved H3 2.55 mm to (123.8, 77.0)
- moved C6 2.50 mm to (113.8, 111.2)
- moved C7 2.50 mm to (117.2, 111.2)
- moved H2 2.50 mm to (123.8, 96.8)
- moved R4 2.49 mm to (115.5, 110.5)
- moved C35 2.18 mm to (99.0, 121.0)
- moved C16 2.00 mm to (115.2, 106.0), turned to 0 degrees
- moved R14 2.00 mm to (116.5, 97.7)
- moved U2 2.00 mm to (116.5, 102.0)
- moved C17 1.95 mm to (117.8, 106.0), turned to 180 degrees
- moved R7 1.82 mm to (88.1, 116.5)
- moved C10 1.49 mm to (88.1, 120.7)
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Connections:
- net Net-(C10-Pad2) renamed /SIMRST
- net Net-(C8-Pad2) renamed /SIMDAT
- net Net-(C9-Pad2) renamed /SIMCLK
- CN3 pad 1: (no net) -> Net-(CN3-Pad1)
- CN3 pad 2: (no net) -> Net-(CN3-Pad2)
- CN3 pad 8: (no net) -> Net-(CN3-Pad8)
- CN4 pad P6: (no net) -> Net-(CN4-PadP6)
- D1 pad 4: (no net) -> Net-(D1-Pad4)
- D1 pad 5: (no net) -> Net-(D1-Pad5)
- D4 pad 4: (no net) -> Net-(D4-Pad4)
- D4 pad 5: (no net) -> Net-(D4-Pad5)
- U1 pad 10: (no net) -> Net-(U1-Pad10)
- U1 pad 11: (no net) -> Net-(U1-Pad11)
- U1 pad 12: (no net) -> Net-(U1-Pad12)
- U1 pad 13: (no net) -> Net-(U1-Pad13)
- U1 pad 46: (no net) -> Net-(U1-Pad46)
- U1 pad 55: (no net) -> Net-(U1-Pad55)
- U1 pad 56: (no net) -> Net-(U1-Pad56)
- U1 pad 57: (no net) -> Net-(U1-Pad57)
- U1 pad 58: (no net) -> Net-(U1-Pad58)
- U1 pad 59: (no net) -> Net-(U1-Pad59)
- U1 pad 60: (no net) -> Net-(U1-Pad60)
- U1 pad 61: (no net) -> Net-(U1-Pad61)
- U1 pad 62: (no net) -> Net-(U1-Pad62)
- U1 pad 63: (no net) -> Net-(U1-Pad63)
- U1 pad 64: (no net) -> Net-(U1-Pad64)
- U1 pad 65: (no net) -> Net-(U1-Pad65)
- U1 pad 66: (no net) -> Net-(U1-Pad66)
- U1 pad 67: (no net) -> Net-(U1-Pad67)
- U1 pad 68: (no net) -> Net-(U1-Pad68)
Routing:
- net GND: track 27.5 -> 109.4 mm
- net GNDD: track 0.00 -> 69.4 mm
- net /SIM1_VDD: track 0.00 -> 32.5 mm, vias 0 -> 2
- net /DBG_RXD: track 0.00 -> 27.0 mm
- net /DBG_TXD: track 0.00 -> 26.6 mm
- net /SIM_RST: track 0.00 -> 21.8 mm
- net /SIMCLK: track 0.00 -> 19.7 mm, vias 0 -> 2
- net /SIMDAT: track 0.00 -> 17.2 mm, vias 0 -> 3
- net /SIM_DAT: track 0.00 -> 16.7 mm
- net /GNSS_VCC_EN: track 0.00 -> 15.9 mm
- net /RST: track 0.00 -> 13.1 mm
- net /ANT_BT: track 0.00 -> 13.0 mm
- net /VDD_EXT: track 0.00 -> 13.0 mm
- net /SIM_CLK: track 0.00 -> 12.9 mm
- net /SIMRST: track 0.00 -> 12.4 mm, vias 0 -> 2
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- added copper zone on F.Cu, net Net-(AE1-Pad2)

Commit message: layout wip
Parts:
- D1: moved to F.Cu
- H3: footprint mc60_fp:Pin_Header_Straight_2x04 -> mc60_fp:Pin_Header_Straight_2x04_Pitch1.27mm
- JP1, JP2: footprint mc60_fp:Pin_Header_Straight_1x03 -> mc60_fp:Pin_Header_Straight_1x03_Pitch1.27mm
- moved H3 52.0 mm to (72.1, 71.1), turned to 180 degrees
- moved JP2 30.0 mm to (94.8, 63.0), turned to 0 degrees
- moved D1 10.0 mm to (85.7, 101.6), turned to 180 degrees
- moved JP1 2.84 mm to (126.3, 89.5)
- moved R14 1.51 mm to (115.0, 97.5), turned to 180 degrees
- moved C1 1.43 mm to (112.4, 89.7), turned to 90 degrees
Connections:
- CN3 pad 1: Net-(CN3-Pad1) -> (no net)
- CN3 pad 2: Net-(CN3-Pad2) -> (no net)
- CN3 pad 8: Net-(CN3-Pad8) -> (no net)
- CN4 pad P6: Net-(CN4-PadP6) -> (no net)
- D1 pad 4: Net-(D1-Pad4) -> (no net)
- D1 pad 5: Net-(D1-Pad5) -> (no net)
- D4 pad 4: Net-(D4-Pad4) -> (no net)
- D4 pad 5: Net-(D4-Pad5) -> (no net)
- H3 pad 5: GND -> VDD
- H3 pad 8: VDD -> GND
- U1 pad 10: Net-(U1-Pad10) -> (no net)
- U1 pad 11: Net-(U1-Pad11) -> (no net)
- U1 pad 12: Net-(U1-Pad12) -> (no net)
- U1 pad 13: Net-(U1-Pad13) -> (no net)
- U1 pad 46: Net-(U1-Pad46) -> (no net)
- U1 pad 55: Net-(U1-Pad55) -> (no net)
- U1 pad 56: Net-(U1-Pad56) -> (no net)
- U1 pad 57: Net-(U1-Pad57) -> (no net)
- U1 pad 58: Net-(U1-Pad58) -> (no net)
- U1 pad 59: Net-(U1-Pad59) -> (no net)
- U1 pad 60: Net-(U1-Pad60) -> (no net)
- U1 pad 61: Net-(U1-Pad61) -> (no net)
- U1 pad 62: Net-(U1-Pad62) -> (no net)
- U1 pad 63: Net-(U1-Pad63) -> (no net)
- U1 pad 64: Net-(U1-Pad64) -> (no net)
- U1 pad 65: Net-(U1-Pad65) -> (no net)
- U1 pad 66: Net-(U1-Pad66) -> (no net)
- U1 pad 67: Net-(U1-Pad67) -> (no net)
- U1 pad 68: Net-(U1-Pad68) -> (no net)
Routing:
- net GND: track 109.4 -> 259.5 mm, vias 0 -> 157
- net VBAT: track 7.97 -> 132.6 mm, vias 0 -> 4
- net VDD: track 7.95 -> 116.7 mm, vias 0 -> 1
- net /VDD_EXT: track 13.0 -> 64.0 mm, vias 0 -> 2
- net /MIC+: track 0.00 -> 42.5 mm
- net /SD_DET>: track 0.00 -> 42.3 mm, vias 0 -> 2
- net /RST: track 13.1 -> 51.3 mm
- net /GSM_PWR_EN: track 0.00 -> 32.9 mm
- net /2V8_SD: track 0.00 -> 31.9 mm, vias 0 -> 3
- net /GNSSVCC: track 7.95 -> 32.7 mm, vias 0 -> 2
- net /PWRKEY: track 0.00 -> 24.4 mm, vias 0 -> 2
- net /SD_DAT: track 0.00 -> 23.8 mm
- net /SD_CLK: track 0.00 -> 22.0 mm, vias 0 -> 2
- net /LOUD_SPKP: track 0.00 -> 20.8 mm
- net GNDREF: track 0.00 -> 20.7 mm
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- added copper zone on B.Cu, net GND

Commit message: layout WIP
Parts:
- added G1: OSHW, mc60_fp:Logo_silk_OSHW_6x6mm, F.Cu at (113.5, 119.5)
- added G2: KiCad, mc60_fp:KiCad-Logo2_6mm_SilkScreen, F.Cu at (119.0, 123.0)
- added G3: LOGO_WL, mc60_fp:Logo-WL3, F.Cu at (91.0, 124.0)
- added H4: ON_OFF, mc60_fp:Pin_Header_Straight_1x03, F.Cu at (72.0, 71.0)
- added SC1: SCREW, mc60_fp:mtg_hole_3mm_vias_2, F.Cu at (126.0, 63.0)
- added SC2: SCREW, mc60_fp:mtg_hole_3mm_vias_2, F.Cu at (72.0, 63.0)
- added SC3: SCREW, mc60_fp:mtg_hole_3mm_vias_2, F.Cu at (126.0, 127.0)
- added SC4: SCREW, mc60_fp:mtg_hole_3mm_vias_2, F.Cu at (96.0, 127.0)
- H3: value CONTROL -> 3V3_EXT; footprint mc60_fp:Pin_Header_Straight_2x04_Pitch1.27mm -> mc60_fp:Pin_Header_Straight_1x03
- moved H3 55.1 mm to (126.0, 82.5), turned to 0 degrees
- moved C35 8.06 mm to (106.0, 125.0), turned to 0 degrees
- moved JP1 2.52 mm to (126.0, 92.0), turned to 180 degrees
- moved H1 2.25 mm to (126.0, 118.8)
- moved CN6 0.85 mm to (78.6, 69.0)
Connections:
- net /MIC+ renamed /MIC_P
- net /MIC- renamed /MIC_N
- CN3 pad 1: (no net) -> Net-(CN3-Pad1)
- CN3 pad 2: (no net) -> Net-(CN3-Pad2)
- CN3 pad 8: (no net) -> Net-(CN3-Pad8)
- CN4 pad P6: (no net) -> Net-(CN4-PadP6)
- D1 pad 4: (no net) -> Net-(D1-Pad4)
- D1 pad 5: (no net) -> Net-(D1-Pad5)
- D4 pad 4: (no net) -> Net-(D4-Pad4)
- D4 pad 5: (no net) -> Net-(D4-Pad5)
- H3 pad 1: /3V3_EXT -> GND
- H3 pad 2: GND -> /3V3_EXT
- H3 pad 3: VDD -> GND
- U1 pad 10: (no net) -> Net-(U1-Pad10)
- U1 pad 11: (no net) -> Net-(U1-Pad11)
- U1 pad 12: (no net) -> Net-(U1-Pad12)
- U1 pad 13: (no net) -> Net-(U1-Pad13)
- U1 pad 46: (no net) -> Net-(U1-Pad46)
- U1 pad 55: (no net) -> Net-(U1-Pad55)
- U1 pad 56: (no net) -> Net-(U1-Pad56)
- U1 pad 57: (no net) -> Net-(U1-Pad57)
- U1 pad 58: (no net) -> Net-(U1-Pad58)
- U1 pad 59: (no net) -> Net-(U1-Pad59)
- U1 pad 60: (no net) -> Net-(U1-Pad60)
- U1 pad 61: (no net) -> Net-(U1-Pad61)
- U1 pad 62: (no net) -> Net-(U1-Pad62)
- U1 pad 63: (no net) -> Net-(U1-Pad63)
- U1 pad 64: (no net) -> Net-(U1-Pad64)
- U1 pad 65: (no net) -> Net-(U1-Pad65)
- U1 pad 66: (no net) -> Net-(U1-Pad66)
- U1 pad 67: (no net) -> Net-(U1-Pad67)
- U1 pad 68: (no net) -> Net-(U1-Pad68)
Routing:
- net /GSM_PWR_EN: track 32.9 -> 5.03 mm
- net VDD: track 116.7 -> 144.0 mm, vias 1 -> 2
- net /3V3_EXT: track 0.00 -> 12.6 mm
- net VBAT: track 132.6 -> 142.1 mm
- net /2V8_SD: track 31.9 -> 36.9 mm
- net GND: track 259.5 -> 264.4 mm
- net Net-(AE1-Pad2): track 1.30 -> 5.34 mm
- net /VCCB: track 23.9 -> 27.6 mm
- net /DBG_TXD: track 26.6 -> 28.8 mm
- net /DBG_RXD: track 27.0 -> 29.3 mm
- net /VDD_EXT: track 64.0 -> 61.8 mm, vias 2 -> 3
- net /MIC_P: track 42.5 -> 44.3 mm
- net /LOUD_SPKP: track 20.8 -> 21.8 mm
- net /MIC_N: track 19.0 -> 19.8 mm
- added copper zone on F.Cu, net VBAT
- added copper zone on F.Cu, net VDD
Other:
- outline, holes or cut-outs redrawn

Commit message: layout WIP
Parts:
- moved H1 13.1 mm to (114.5, 125.0)
- moved G1 11.9 mm to (125.4, 119.4)
- moved C36 4.13 mm to (102.5, 118.2), turned to 90 degrees
- moved AE1 3.98 mm to (126.6, 110.8)
- moved C6 3.43 mm to (117.0, 112.5)
- moved C7 3.43 mm to (120.5, 112.5)
- moved R4 3.43 mm to (118.7, 111.7)
- moved C1 2.30 mm to (114.5, 88.8), turned to 0 degrees
- moved D2 2.25 mm to (122.8, 88.1)
- moved Q1 2.25 mm to (118.5, 88.1)
- moved R8 2.25 mm to (121.2, 88.1)
- moved C29 2.00 mm to (116.0, 67.0)
- moved C30 2.00 mm to (116.0, 80.0)
- moved S1 0.60 mm to (74.2, 109.8)
- moved C35 0.50 mm to (106.0, 125.5)
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Routing:
- net /DBG_RXD: track 29.3 -> 21.0 mm
- net /DBG_TXD: track 28.8 -> 22.7 mm
- net GND: track 264.4 -> 269.3 mm, vias 157 -> 159
- net /VCCB: track 27.6 -> 23.7 mm
- net /ANT_BT: track 13.2 -> 16.7 mm
- net VBAT: track 142.1 -> 144.6 mm
- net /NETLIGHT: track 16.0 -> 18.2 mm
- net VDD: track 144.0 -> 141.8 mm
- net /VDD_EXT: track 61.8 -> 63.6 mm
- net /PWRKEY: track 24.4 -> 25.0 mm
- net /SD_DET>: track 41.9 -> 42.5 mm
- net /RST: track 50.9 -> 51.5 mm
- net GNDD: track 79.2 -> 78.6 mm
- net Net-(AE1-Pad2): track 5.34 -> 5.93 mm
- net /GNSS_VCC_EN: track 15.9 -> 15.4 mm
